File: Modbus-RJ45-Breakout.kicad_sch (KiCad schematic)
At the start: 145 parts, among them J1 RJ45_Weidmueller_2562920000, J2 RJ45_Weidmueller_2562920000, J3 Bus_2, J4 BUS_1, J5 USB_B_Mini, J6 2X04, J7 WAGO 2734-104, Q1 BSP250, U1 FT2232D, U2 WE-TVS-82400102, U3 MAX485E, U4 ADM2687E, U5 93LC46B, U6 WE-TVS-82400102, U7 MAX485E, U8 ADM2687E, Y1 6MHz

Commit message: Version bump 1.0.0
Parts:
- DRA1, J7: footprint (none) -> the78mole:Dummy_0
- J8: value (none) -> WAGO 2734-104; footprint (none) -> the78mole:Dummy_0
Changed lines of the file:
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@@
   (title_block
     (title "Modbus-RJ45-Breakout")
-    (date "2023-04-24")
-    (rev "0.0.1")
+    (date "2023-06-02")
+    (rev "1.0.0")
     (company "the78mole")
   )
@@
     (in_bom yes) (on_board yes)
     (property "Reference" "J8" (id 0) (at 388.62 80.01 0))
-    (property "Value" "" (id 1) (at 388.62 82.55 0))
-    (property "Footprint" "" (id 2) (at 387.985 90.17 0)
+    (property "Value" "WAGO 2734-104" (id 1) (at 388.62 82.55 0))
+    (property "Footprint" "the78mole:Dummy_0" (id 2) (at 387.985 90.17 0)
       (effects (font (size 1.27 1.27)) hide)
     )
@@
     (property "Reference" "DRA1" (id 0) (at 361.95 203.2 0))
     (property "Value" "APRA 449-440-45" (id 1) (at 361.95 205.74 0))
-    (property "Footprint" "" (id 2) (at 361.95 215.9 0)
+    (property "Footprint" "the78mole:Dummy_0" (id 2) (at 361.95 215.9 0)
       (effects (font (size 1.27 1.27)) hide)
     )
@@
     (property "Reference" "J7" (id 0) (at 388.62 20.955 0))
     (property "Value" "WAGO 2734-104" (id 1) (at 388.62 23.495 0))
-    (property "Footprint" "" (id 2) (at 387.985 31.115 0)
+    (property "Footprint" "the78mole:Dummy_0" (id 2) (at 387.985 31.115 0)
       (effects (font (size 1.27 1.27)) hide)
     )
